File: pcb/generic-top-test-jig.kicad_pcb (KiCad board)
At the start: 2 copper layers, 45 x 39.2 mm, 37 parts, among them P1 CONN_01X16, U1 74HC4051, U2 74HC4067, U3 74HC4067, U4 74HC4067, U5 74HC4067

Commit message: Add license information to many files. PCB design files are CC-BY and code is MIT license.
Other:
- board text added: "Copyright 2016 Chickadee Tech LLC, <add attributions here> This work is licensed under the Creative Commons Attribution 4.0 International License. To view a copy of this license, visit http://creativecommons.org/licenses/by/4.0/ or send a letter to Creative Commons, PO Box 1866, Mountain View, CA 94042, USA."
- board text added: "Remove all Chickadee Tech LLC trademarks before making your own board. The Chickadee logo and Polystack logo are owned by Chickadee Tech LLC. You may license the Polystack logo for free by emailing support@chickadee.tech and receiving express written permission from Chickadee Tech LLC."
- board text added: "The gear logo is a mark designating open source hardware. Remove it if your design does not comply with the open source hardware definition."
Changed lines of the file:
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@@
     (area 118.127143 74.1 268.690476 178)
     (thickness 1.6)
-    (drawings 33)
+    (drawings 39)
     (tracks 1925)
     (zones 0)
@@
     (40 Dwgs.User user)
     (41 Cmts.User user)
-    (42 Eco1.User user hide)
-    (43 Eco2.User user hide)
+    (42 Eco1.User user)
+    (43 Eco2.User user)
     (44 Edge.Cuts user)
     (45 Margin user)
@@
       (xy 4.672239 -0.694521)) (layer B.SilkS) (width 0))
   )
+  (gr_line (start 135.48 98.02) (end 176.58 124.41) (layer Cmts.User) (width 0.2))
+  (gr_text "The gear logo is a mark designating open\nsource hardware. Remove it if your design\ndoes not comply with the open source\nhardware definition." (at 177.31 124.77) (layer Cmts.User)
+    (effects (font (size 1.5 1.5) (thickness 0.3)) (justify left))
+  )
+  (gr_line (start 105.57 108.82) (end 154.84 127.04) (layer Cmts.User) (width 0.2))
+  (gr_line (start 136.73 98.07) (end 105.57 108.82) (layer Cmts.User) (width 0.2))
+  (gr_text "Remove all Chickadee Tech LLC trademarks\nbefore making your own board. The\nChickadee logo and Polystack logo\nare owned by Chickadee Tech LLC.\n\nYou may license the Polystack logo for\nfree by emailing support@chickadee.tech\nand receiving express written permission\nfrom Chickadee Tech LLC." (at 63.87 109.7) (layer Cmts.User)
+    (effects (font (size 1.5 1.5) (thickness 0.3)) (justify left))
+  )
+  (gr_text "Copyright 2016 Chickadee Tech LLC, <add attributions here>\n\nThis work is licensed under the Creative Commons Attribution 4.0 International License.\nTo view a copy of this license, visit http://creativecommons.org/licenses/by/4.0/\nor send a letter to Creative Commons, PO Box 1866, Mountain View, CA 94042, USA." (at 178.57 174.02) (layer Cmts.User)
+    (effects (font (size 1.5 1.5) (thickness 0.3)) (justify left))
+  )
   (gr_text 48-63 (at 161.8 122.7) (layer F.SilkS)
     (effects (font (size 1 1) (thickness 0.15)))
@@
   )
   (gr_arc (start 172.25 92.75) (end 172.25 90) (angle 90) (layer Edge.Cuts) (width 0.15))
-  (gr_text "Try to keep components outside\nthe yellow rings. They designate\n8mm diameter washers that may\nbe used to separate boards." (at 167.5 100.9) (layer Eco2.User)
+  (gr_text "Try to keep components outside\nthe yellow rings. They designate\n8mm diameter washers that may\nbe used to separate boards." (at 177.11 100.89) (layer Eco2.User)
     (effects (font (size 1.5 1.5) (thickness 0.25)) (justify left))
   )
@@
   (gr_line (start 175 92.75) (end 175 126.5) (angle 90) (layer Edge.Cuts) (width 0.15))
   (gr_line (start 132.75 90) (end 172.25 90) (angle 90) (layer Edge.Cuts) (width 0.15))
-  (gr_text generic-top-test-jig (at 187.25 174.25) (layer Cmts.User)
-    (effects (font (size 5 5) (thickness 0.5)) (justify left))
+  (gr_text generic-top-test-jig (at 187.05 189.65) (layer Cmts.User)
+    (effects (font (size 3 3) (thickness 0.5)) (justify left))
   )
   (segment (start 138.228709 113.821291) (end 138 114.05) (width 0.254) (layer B.Cu) (net 0))
